File: thumb-pcb/kinesis-thumb-pcb.kicad_pcb (KiCad board)
At the start: 2 copper layers, 77 x 88 mm, 33 parts, among them J1 Conn_01x10

Commit message: Update files and readme
Parts:
- D1, D10, D11, D12, D2, D3, D4, D5, D6, D7, D8, D9: footprint Diode_SMD:D_SOD-323_HandSoldering -> keyboard_parts:D_SOD123W_hand
- moved D5 14.3 mm to (187.3, 73.0), turned to 180 degrees
- moved D6 14.3 mm to (187.3, 92.1), turned to 180 degrees
- moved D8 14.3 mm to (187.3, 73.0)
- moved D9 14.3 mm to (187.3, 92.1)
- moved D4 14.3 mm to (187.3, 54.0), turned to 180 degrees
- moved D7 14.3 mm to (187.3, 54.0)
- moved D1 14.3 mm to (206.4, 54.0), turned to 180 degrees
- moved D10 14.3 mm to (206.4, 54.0)
- moved D11 14.3 mm to (206.4, 82.5)
- moved D12 14.3 mm to (225.4, 82.5)
- moved D2 14.3 mm to (206.4, 82.5), turned to 180 degrees
- moved D3 14.3 mm to (225.4, 82.5), turned to 180 degrees
Connections:
- D10 pad 1: /COL_L5 -> /ROW_8
- D11 pad 1: /COL_L6 -> /ROW_7
- D12 pad 1: /ROW_5 -> /ROW_6
- D3 pad 1: /COL_R5 -> /ROW_3
- D5 pad 1: /COL_R5 -> /ROW_3
- D8 pad 1: /COL_L5 -> /ROW_8
- D9 pad 1: /ROW_5 -> /ROW_6
- J1 pad 6: /ROW_9 -> unconnected-(J1-Pin_6-Pad6)
- J1 pad 7: /COL_R6 -> unconnected-(J1-Pin_7-Pad7)
- J1 pad 8: /COL_R5 -> /ROW_3
Routing:
- net /ROW_3: track 0.00 -> 116.5 mm, vias 0 -> 3
- net /ROW_6: track 0.00 -> 112.8 mm, vias 0 -> 1
- net /ROW_5: track 132.7 -> 50.4 mm, vias 3 -> 2
- net /COL_R5: track 143.0 -> 69.1 mm, vias 3 -> 1
- net /ROW_8: track 0.00 -> 69.9 mm, vias 0 -> 1
- net /ROW_7: track 0.00 -> 62.0 mm, vias 0 -> 1
- net /COL_L5: track 111.4 -> 55.9 mm, vias 3 -> 1
- net /COL_L6: track 140.5 -> 87.8 mm, vias 2 -> 0
- net /ROW_9: track 10.7 -> 35.1 mm
- net /ROW_2: track 58.9 -> 71.2 mm
- net /ROW_4: track 70.8 -> 81.9 mm, vias 2 -> 3
- net Net-(D8-A): track 4.90 -> 10.2 mm
- net Net-(D7-A): track 4.90 -> 10.2 mm
- net Net-(D9-A): track 4.90 -> 10.2 mm
- net Net-(D12-A): track 4.98 -> 10.2 mm
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Other:
- board text added: "Pillz Mod thumb cluster LEFT Rev 2 github.com/dcpedit/pillzmod"
- board text added: "Pillz Mod thumb cluster RIGHT Rev 2 github.com/dcpedit/pillzmod"
- board text removed: "Pillz Mod thumb cluster left Rev 1 github.com/dcpedit/pillzmod"
- board text removed: "Pillz Mod thumb cluster right Rev 1 github.com/dcpedit/pillzmod"
