File: pcb/kicad_port.kicad_pcb (KiCad board)
At the start: 2 copper layers, 100 x 86 mm, 25 parts, among them J1 Conn_01x13, J2 Conn_01x13, J3 Conn_01x13, J4 Conn_01x13, J5 Conn_01x10, J6 Conn_01x10, J7 Conn_01x13, J8 Conn_01x13, M1 MountingHole_6.4mm_M6, M3 MountingHole_4.3mm_M4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

Commit message: pro-micro support
Parts:
- added BZ1: Buzzer, Buzzer_Beeper:Buzzer_TDK_PS1240P02BT_D12.2mm_H6.5mm, B.Cu at (107.5, 82.9)
- added D6: D_Small, Keebio-Parts:Diode-dual, B.Cu at (165.1, 57.0)
- added D7: D_Small, Keebio-Parts:Diode-dual, B.Cu at (168.3, 57.0)
- added D8: D_Small, Keebio-Parts:Diode-dual, B.Cu at (171.4, 57.0)
- added H1: mounting pad, MountingHole:MountingHole_2mm, B.Cu at (150.0, 60.0)
- added J10: Conn_01x02, Connector_PinHeader_2.54mm:PinHeader_1x02_P2.54mm_Vertical, B.Cu at (116.6, 75.7)
- added J9: Conn_01x04, Connector_PinHeader_2.54mm:PinHeader_1x04_P2.54mm_Vertical, B.Cu at (124.1, 54.1)
- added R5: R_22K, Keebio-Parts:Resistor-Hybrid, B.Cu at (108.5, 89.5)
- D5, R1, R2, R3, R4: moved to B.Cu
- moved D5 2.99 mm to (161.9, 57.0)
Connections:
- D5 pad 1: /ROW_0 -> /ROW_EQL
- SW1 pad S2: /COL_4 -> /COL_5
- U1 pad 22: unconnected-(U1-PC13-Pad22) -> /SOL
- U1 pad 40: unconnected-(U1-5V-Pad40) -> +5V
- U1 pad 7: unconnected-(U1-PA10-Pad7) -> /BUZ
Routing:
- net /ROW_EQL: track 34.3 -> 110.0 mm, vias 0 -> 1
- net /ROW_2: track 61.7 -> 135.1 mm, vias 1 -> 2
- net /ROW_1: track 36.0 -> 108.4 mm, vias 0 -> 1
- net +5V: track 0.00 -> 71.6 mm
- net /BUZ: track 0.00 -> 60.4 mm, vias 0 -> 1
- net /COL_6: track 169.1 -> 221.3 mm, vias 1 -> 3
- net Net-(D8-A): track 0.00 -> 41.9 mm, vias 0 -> 1
- net /ROW_0: track 75.3 -> 34.4 mm
- net Net-(D7-A): track 0.00 -> 40.7 mm, vias 0 -> 1
- net Net-(D6-A): track 0.00 -> 39.9 mm
- net /COL_5: track 249.1 -> 278.8 mm, vias 1 -> 4
- net /COL_4: track 227.6 -> 200.3 mm
- net /SOL: track 0.00 -> 7.90 mm
- net /ROW_5: track 81.6 -> 88.9 mm, vias 2 -> 4
- net Net-(D5-A): track 8.44 -> 14.0 mm
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Other:
- board text added: "Pillz Mod github.com/dcpedit/pillzmod by dcpedit (Rev 2)"
- board text removed: "Pillz Mod github.com/dcpedit/pillzmod by dcpedit (Rev 1)"
