File: pcb/kicad_port.kicad_sch (KiCad schematic)
At the start: 20 parts, among them J1 Conn_01x13, J2 Conn_01x13, J3 Conn_01x13, J4 Conn_01x13, J5 Conn_01x10, J6 Conn_01x10, J7 Conn_01x13, J8 Conn_01x13, SW1 RotaryEncoder_Switch, U1 YAAJ_WeAct_BlackPill_Part_Lik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

Commit message: pro-micro support
Parts:
- added BZ1: Buzzer, symbol Device:Buzzer
- added D6, D7, D8: D_Small, symbol Device:D_Small
- added J10: Conn_01x02, symbol Connector_Generic:Conn_01x02
- added J9: Conn_01x04, symbol Connector_Generic:Conn_01x04
- added R5: R_22K, Keebio-Parts:Resistor, symbol Device:R_Small
Connections:
- net COL_4: no longer SW1.S2
- net COL_5: now also SW1.S2
- net COL_6: now also J9.1 (Pin_1)
- net GND: now also BZ1.2 (+)
- net ROW_0: no longer D5.1 (K)
- net ROW_1: now also D7.1 (K)
- net ROW_2: now also D8.1 (K)
- net ROW_EQL: now also D5.1 (K), D6.1 (K)
- net SOL: now reaches U1.22 (PC13)
- net SOL: now also J10.2 (Pin_2)
- net +5V: now reaches U1.40 (5V)
- net +5V: now also J10.1 (Pin_1), R5.1
- net BUZ: now reaches U1.7 (PA10)
- net BUZ: now also BZ1.1 (-), R5.2
- new net: D7.2 (A), J9.3 (Pin_3)
- new net: D8.2 (A), J9.4 (Pin_4)
- new net: D6.2 (A), J9.2 (Pin_2)
- no-connect marks 36 -> 33
Other:
- note added: "PA13 PA14"
- note added: "PEDAL_GND"
- note added: "PEDAL_SW1"
- note added: "PEDAL_SW2"
- note added: "PEDAL_SW3"
