File: pcb-pro/pcb-pro.kicad_pcb (KiCad board)
At the start: 2 copper layers, 100 x 86 mm, 47 parts, among them J1 Conn_01x13, J10 Extra, J2 Conn_01x13, J3 Conn_01x13, J4 Conn_01x13, J5 Conn_01x10, J6 Conn_01x10, J7 Conn_01x13, J8 Conn_01x13, J9 Conn_01x04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

Commit message: Cleanup
Parts:
- added SW1: RESET, Button_Switch_SMD:SW_SPST_SKQG_WithoutStem, B.Cu at (140.5, 61.1)
Connections:
- U1 pad 22: unconnected-(U1-RST-Pad22) -> /RESET
Routing:
- net /RESET: track 0.00 -> 29.8 mm
Other:
- board text added: "Pillz Mod Pro github.com/dcpedit/pillzmod by dcpedit (Rev 2)"
- board text removed: "Pillz Mod Pro github.com/dcpedit/pillzmod by dcpedit (Rev 1)"

Commit message: Update readme with pro
Parts:
- moved BZ1 4.93 mm to (107.5, 87.8)
Routing:
- net /BUZ: track 31.7 -> 26.8 mm
Changed lines of the file:
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@@
 	(footprint "Buzzer_Beeper:Buzzer_TDK_PS1240P02BT_D12.2mm_H6.5mm"
 		(layer "B.Cu")
-		(at 107.5 82.870785 90)
+		(at 107.5 87.804 90)
 		(descr "Buzzer, D12.2mm height 6.5mm, https://product.tdk.com/info/en/catalog/datasheets/piezoelectronic_buzzer_ps_en.pdf")
 		(tags "buzzer")
@@
 	)
 	(segment
-		(start 106.25 82.870785)
-		(end 103.381698 85.739087)
-		(width 0.25)
-		(layer "B.Cu")
-		(net 62)
-	)
-	(segment
-		(start 103.381698 88.138)
-		(end 103.381698 94.996)
-		(width 0.25)
-		(layer "B.Cu")
-		(net 62)
-	)
-	(segment
-		(start 107.5 82.870785)
-		(end 106.25 82.870785)
+		(start 103.381698 90.672302)
+		(end 103.381698 95.737)
 		(width 0.25)
 		(layer "B.Cu")
@@
 	)
 	(segment
-		(start 103.381698 94.996)
-		(end 103.381698 95.737)
+		(start 107.5 87.804)
+		(end 106.25 87.804)
 		(width 0.25)
 		(layer "B.Cu")
@@
 	)
 	(segment
-		(start 103.381698 85.739087)
-		(end 103.381698 88.138)
+		(start 106.25 87.804)
+		(end 103.381698 90.672302)
 		(width 0.25)
 		(layer "B.Cu")
