File: pcb-pro/pcb-pro.kicad_sch (KiCad schematic)
At the start: 41 parts, among them J1 Conn_01x13, J10 Extra, J2 Conn_01x13, J3 Conn_01x13, J4 Conn_01x13, J5 Conn_01x10, J6 Conn_01x10, J7 Conn_01x13, J8 Conn_01x13, J9 Conn_01x04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

Commit message: Cleanup
Parts:
- added JP2: SolderJumper_2_Open, Jumper:SolderJumper-2_P1.3mm_Open_RoundedPad1.0x1.5mm, symbol Jumper:SolderJumper_2_Open
- added SW1: RESET, symbol Switch:SW_SPST
Connections:
- net EXTRA: now also JP2.1 (A)
- net GND: now also SW1.2 (B); no longer U1.3 (GND)
- net RESET: now reaches U1.22 (RST)
- net RESET: now also SW1.1 (A)
- new net D10: JP2.2 (B), U1.3 (GND)
- no-connect marks 27 -> 26
Other:
- note added: "/0"
- note added: "/1"
- note added: "18/"
- note added: "19/"
- note added: "20/"
- note added: "21/"
- moved on the sheet: JP1

Commit message: Update readme with pro
Parts:
- removed JP2: SolderJumper_2_Open, Jumper:SolderJumper-2_P1.3mm_Open_RoundedPad1.0x1.5mm, symbol Jumper:SolderJumper_2_Open
Connections:
- net D10 is gone; now on net GND: U1.3 (GND)
Changed lines of the file:
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@@
 	)
 	(junction
+		(at 99.06 34.29)
+		(diameter 0)
+		(color 0 0 0 0)
+	)
+	(junction
 		(at 256.54 125.73)
 		(diameter 0)
@@
 	(wire
 		(pts
-			(xy 91.44 34.29) (xy 115.57 34.29)
+			(xy 91.44 34.29) (xy 99.06 34.29)
+		)
+		(stroke
+			(width 0)
+			(type default)
+		)
+	)
+	(wire
+		(pts
+			(xy 99.06 34.29) (xy 115.57 34.29)
 		)
 		(stroke
@@
 	(wire
 		(pts
-			(xy 171.45 76.2) (xy 184.15 76.2)
-		)
-		(stroke
-			(width 0)
-			(type default)
-		)
-	)
-	(wire
-		(pts
 			(xy 256.54 125.73) (xy 256.54 128.27)
 		)
@@
 	(wire
 		(pts
+			(xy 99.06 31.75) (xy 99.06 34.29)
+		)
+		(stroke
+			(width 0)
+			(type default)
+		)
+	)
+	(wire
+		(pts
 			(xy 207.01 74.93) (xy 209.55 74.93)
 		)
@@
 	(wire
 		(pts
-			(xy 163.83 76.2) (xy 153.67 76.2)
-		)
-		(stroke
-			(width 0)
-			(type default)
-		)
-	)
-	(wire
-		(pts
 			(xy 256.54 105.41) (xy 256.54 107.95)
 		)
@@
 		)
 	)
-	(label "D10"
-		(at 184.15 76.2 180)
-		(fields_autoplaced yes)
-		(effects
-			(font
-				(size 1.27 1.27)
-			)
-			(justify right bottom)
-		)
-	)
 	(label "ROW_13"
 		(at 207.01 22.86 180)
@@
 		)
 	)
-	(label "EXTRA"
-		(at 153.67 76.2 0)
-		(fields_autoplaced yes)
-		(effects
-			(font
-				(size 1.27 1.27)
-			)
-			(justify left bottom)
-		)
-	)
 	(label "ROW_10"
 		(at 238.76 130.81 0)
@@
 		)
 	)
-	(label "D10"
-		(at 99.06 31.75 0)
-		(fields_autoplaced yes)
-		(effects
-			(font
-				(size 1.27 1.27)
-			)
-			(justify left bottom)
-		)
-	)
 	(label "LATCH"
 		(at 161.29 54.61 180)
@@
 	)
 	(symbol
-		(lib_id "Jumper:SolderJumper_2_Open")
-		(at 167.64 76.2 0)
-		(unit 1)
-		(exclude_from_sim no)
-		(in_bom yes)
-		(on_board yes)
-		(dnp no)
-		(property "Reference" "JP2"
-			(at 167.64 78.74 0)
-			(effects
-				(font
-					(size 1.27 1.27)
-				)
-			)
-		)
-		(property "Value" "SolderJumper_2_Open"
-			(at 167.64 73.3044 0)
-			(effects
-				(font
-					(size 1.27 1.27)
-				)
-				(hide yes)
-			)
-		)
-		(property "Footprint" "Jumper:SolderJumper-2_P1.3mm_Open_RoundedPad1.0x1.5mm"
-			(at 167.64 76.2 0)
-			(effects
-				(font
-					(size 1.27 1.27)
-				)
-				(hide yes)
-			)
-		)
-		(property "Datasheet" "~"
-			(at 167.64 76.2 0)
-			(effects
-				(font
-					(size 1.27 1.27)
-				)
-				(hide yes)
-			)
-		)
-		(property "Description" ""
-			(at 167.64 76.2 0)
-			(effects
-				(font
-					(size 1.27 1.27)
-				)
-				(hide yes)
-			)
-		)
-		(pin "1"
-		)
-		(pin "2"
-		)
-		(instances
-			(project "pcb-pro"
-				(path "/2f5297a0-6822-492a-a296-0cbef0b8cf70"
-					(reference "JP2")
-					(unit 1)
-				)
-			)
-		)
-	)
-	(symbol
 		(lib_id "Device:R")
 		(at 252.73 113.03 90)
@@
 					(size 1.27 1.27)
 				)
+				(hide yes)
 			)
 		)
